File: elec/obc/obc.kicad_sch (KiCad schematic)
At the start: 26 parts, among them J1 Conn_01x02_Pin, J2 Conn_01x02_Pin, U1 STM32G474RBT3, U2 BMP585, U3 H3LIS331DLTR, U4 SAM_M10Q_00B, U5 TMP1075D

Commit message: yes
Parts:
- added J3: IDC_6P, Bluesat:IDC6, symbol Bluesat:IDC_6P
Changed lines of the file:
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@@
+	)
+	(symbol
+		(lib_id "Bluesat:IDC_6P")
+		(at 156.21 142.24 0)
+		(unit 1)
+		(body_style 1)
+		(exclude_from_sim no)
+		(in_bom yes)
+		(on_board yes)
+		(in_pos_files yes)
+		(dnp no)
+		(fields_autoplaced yes)
+		(property "Reference" "J3"
+			(at 156.845 133.35 0)
+			(show_name no)
+			(do_not_autoplace no)
+			(effects
+				(font
+					(size 1.27 1.27)
+				)
+			)
+		)
+		(property "Value" "IDC_6P"
+			(at 156.845 135.89 0)
+			(show_name no)
+			(do_not_autoplace no)
+			(effects
+				(font
+					(size 1.27 1.27)
+				)
+			)
+		)
+		(property "Footprint" "Bluesat:IDC6"
+			(at 156.21 142.24 0)
+			(hide yes)
+			(show_name no)
+			(do_not_autoplace no)
+			(effects
+				(font
+					(size 1.27 1.27)
+				)
+			)
+		)
+		(property "Datasheet" "Bluesat OWR docs: standard/electrical/device#debugging"
+			(at 156.21 142.24 0)
+			(hide yes)
+			(show_name no)
+			(do_not_autoplace no)
+			(effects
+				(font
+					(size 1.27 1.27)
+				)
+			)
+		)
+		(property "Description" "6-pin IDC MCU debug header (socket for debuggers)"
+			(at 156.21 142.24 0)
+			(hide yes)
+			(show_name no)
+			(do_not_autoplace no)
+			(effects
+				(font
+					(size 1.27 1.27)
+				)
+			)
+		)
+		(pin "1"
+		)
+		(pin "2"
+		)
+		(pin "3"
+		)
+		(pin "4"
+		)
+		(pin "5"
+		)
+		(pin "6"
+		)
+		(instances
+			(project "obc"
+				(path "/5ac93bd7-40e0-43d4-a63b-ad562fa6459a"
+					(reference "J3")
+					(unit 1)
+				)
+			)
+		)
 	)
 	(symbol
